File: PCB Design/WinterPercussion/WinterPercussion.kicad_pcb (KiCad board)
At the start: 2 copper layers, 55.9 x 59 mm, 6 parts, among them J1 SDS-50J, U1 H11L1M, U2 ESP32-DevKitC

Commit message: Diode UPdate
Parts:
- D1: footprint Diode_THT:D_T-1_P5.08mm_Horizontal -> Diode_THT:D_DO-41_SOD81_P10.16mm_Horizontal
- moved D1 0.08 mm to (137.2, 71.1)
Connections:
- D1 pad 1: Net-(D1-Pad1) -> Net-(D1-K)
- D1 pad 2: Net-(D1-Pad2) -> Net-(D1-A)
- R1 pad 1: Net-(D1-Pad2) -> Net-(D1-K)
- U1 pad 1: Net-(D1-Pad2) -> Net-(D1-K)
- U1 pad 2: Net-(D1-Pad1) -> Net-(D1-A)
Routing:
- net Net-(D1-K): track 0.00 -> 31.9 mm
- net Net-(D1-Pad1): track 30.0 -> 0.00 mm
- net Net-(D1-Pad2): track 25.8 -> 0.00 mm
- net Net-(D1-A): track 0.00 -> 16.5 mm

Commit message: Add files via upload
Parts:
- D1: footprint Diode_THT:D_DO-41_SOD81_P10.16mm_Horizontal -> Diode_THT:D_DO-201AD_P15.24mm_Horizontal
- moved D1 2.54 mm to (137.2, 68.6)
Routing:
- net Net-(J1-Pad5): track 16.5 -> 23.9 mm
- net GND: track 46.8 -> 41.9 mm, vias 0 -> 1
- net Net-(R1-Pad1): track 31.9 -> 33.4 mm
Other:
- board text added: "Pin 1"
