File: PCB Design/WinterPercussion/WinterPercussion.kicad_sch (KiCad schematic)
At the start: 2 parts

Commit message: Board Design
Parts:
- added D1: DIODE, Diode_THT:D_T-1_P5.08mm_Horizontal, symbol pspice:DIODE
- added R1: 220Ω, Resistor_THT:R_Axial_DIN0207_L6.3mm_D2.5mm_P7.62mm_Horizontal, symbol Device:R_US
- added R2: 10kΩ, Resistor_THT:R_Axial_DIN0207_L6.3mm_D2.5mm_P7.62mm_Horizontal, symbol Device:R_US
- added R3: 470Ω, Resistor_THT:R_Axial_DIN0207_L6.3mm_D2.5mm_P7.62mm_Horizontal, symbol Device:R_US
- added U1: 6N138, OptoCoupler:DIP762W50P254L1018H450Q8, symbol Isolator:6N138
- gave numbers to parts that had none: 2
Connections:
- net at J1.4: now also R1.2
- net at J1.5: now also D1.1 (K), U1.3 (C2)
- net +5V: now reaches U2.19 (5V)
- net +5V: now also R3.1, U1.8 (VCC)
- net GND: now reaches U2.38 (GND)
- net GND: now also R2.2, U1.5 (GND)
- new net: D1.2 (A), R1.1, U1.2 (C1)
- new net: R2.1, U1.7 (VO1)
- new net ESP_PIN: R3.2, U1.6 (VO2)
- no-connect marks 0 -> 40
Other:
- moved on the sheet: J1, U2

Commit message: Updated with Pin16 from Mark
Connections:
- net ESP_PIN: now also U2.27 (GPIO16)
- no-connect marks 40 -> 39
Changed lines of the file:
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@@
   (no_connect (at 248.92 102.87))
   (no_connect (at 248.92 100.33))
-  (no_connect (at 248.92 97.79))
   (no_connect (at 248.92 90.17))
   (no_connect (at 248.92 87.63))
@@
     (stroke (width 0) (type default) (color 0 0 0 0))
   )
+  (wire (pts (xy 248.92 97.79) (xy 259.08 97.79))
+    (stroke (width 0) (type default) (color 0 0 0 0))
+  )
   (wire (pts (xy 148.59 64.77) (xy 161.29 64.77))
     (stroke (width 0) (type default) (color 0 0 0 0))
@@
       (effects (font (size 1.27 1.27)) (justify left) hide)
     )
+  )
+  (global_label "ESP_PIN" (shape input) (at 259.08 97.79 0) (fields_autoplaced)
+    (effects (font (size 1.27 1.27)) (justify left))
+    (property "Intersheet References" "${INTERSHEET_REFS}" (id 0) (at 269.2945 97.7106 0)
+      (effects (font (size 1.27 1.27)) (justify left) hide)
+    )

Commit message: Updated KiCad Docs
Parts:
- removed R2: 10kΩ, Resistor_THT:R_Axial_DIN0207_L6.3mm_D2.5mm_P7.62mm_Horizontal, symbol Device:R_US
- removed R3: 470Ω, Resistor_THT:R_Axial_DIN0207_L6.3mm_D2.5mm_P7.62mm_Horizontal, symbol Device:R_US
- removed U1: 6N138, OptoCoupler:DIP762W50P254L1018H450Q8, symbol Isolator:6N138
- added R2: 270Ω, Resistor_THT:R_Axial_DIN0207_L6.3mm_D2.5mm_P7.62mm_Horizontal, symbol Device:R_Small_US
- added U1: H11L1M, Opto:H11L1M, symbol OptoCoupler:H11L1M
Connections:
- net +5V: now also R2.1, U1.6 (VCC)
- net ESP_PIN: now also R2.2, U1.4 (VO)
- net GND: now also U1.5 (GND)
- net at D1.2 (A), R1.1: now also U1.1 (ANODE)
- net at D1.1 (K), J1.5: now also U1.2 (CATHODE)
Other:
- moved on the sheet: D1, J1, R1

Commit message: Changed to 3.3v
Connections:
- net +3V3: now reaches U2.1 (3V3)
- net +3V3: now also R2.1, U1.6 (VCC)
- removed net +5V: R2.1, U1.6 (VCC), U2.19 (5V)
Changed lines of the file:
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@@
   (no_connect (at 179.07 97.79))
   (no_connect (at 179.07 100.33))
-  (no_connect (at 179.07 69.85))
+  (no_connect (at 179.07 115.57))
   (no_connect (at 179.07 110.49))
   (no_connect (at 179.07 113.03))
@@
     (stroke (width 0) (type default) (color 0 0 0 0))
   )
-  (wire (pts (xy 165.1 115.57) (xy 179.07 115.57))
+  (wire (pts (xy 176.53 69.85) (xy 179.07 69.85))
     (stroke (width 0) (type default) (color 0 0 0 0))
   )
@@
       (effects (font (size 1.27 1.27)) (justify left) hide)
     )
+  )
+  (symbol (lib_id "power:+3V3") (at 130.81 69.85 0) (unit 1)
+    (in_bom yes) (on_board yes) (fields_autoplaced)
+    (property "Reference" "#PWR0101" (id 0) (at 130.81 73.66 0)
+      (effects (font (size 1.27 1.27)) hide)
+    )
+    (property "Value" "+3V3" (id 1) (at 130.81 64.77 0))
+    (property "Footprint" "" (id 2) (at 130.81 69.85 0)
+      (effects (font (size 1.27 1.27)) hide)
+    )
+    (property "Datasheet" "" (id 3) (at 130.81 69.85 0)
+      (effects (font (size 1.27 1.27)) hide)
+    )
+    (pin "1")
   )
   (symbol (lib_id "Device:R_Small_US") (at 146.05 72.39 0) (unit 1)
@@
     (pin "9")
   )
-  (symbol (lib_id "power:+5V") (at 130.81 69.85 0) (unit 1)
-    (in_bom yes) (on_board yes) (fields_autoplaced)
-    (property "Reference" "#PWR01" (id 0) (at 130.81 73.66 0)
-      (effects (font (size 1.27 1.27)) hide)
-    )
-    (property "Value" "+5V" (id 1) (at 130.81 64.77 0))
-    (property "Footprint" "" (id 2) (at 130.81 69.85 0)
-      (effects (font (size 1.27 1.27)) hide)
-    )
-    (property "Datasheet" "" (id 3) (at 130.81 69.85 0)
+  (symbol (lib_id "power:+3V3") (at 176.53 69.85 0) (unit 1)
+    (in_bom yes) (on_board yes) (fields_autoplaced)
+    (property "Reference" "#PWR?" (id 0) (at 176.53 73.66 0)
+      (effects (font (size 1.27 1.27)) hide)
+    )
+    (property "Value" "+3V3" (id 1) (at 176.53 64.77 0))
+    (property "Footprint" "" (id 2) (at 176.53 69.85 0)
+      (effects (font (size 1.27 1.27)) hide)
+    )
+    (property "Datasheet" "" (id 3) (at 176.53 69.85 0)
       (effects (font (size 1.27 1.27)) hide)
     )
@@
     (pin "1")
   )
-  (symbol (lib_id "power:+5V") (at 165.1 115.57 0) (unit 1)
-    (in_bom yes) (on_board yes) (fields_autoplaced)
-    (property "Reference" "#PWR03" (id 0) (at 165.1 119.38 0)
-      (effects (font (size 1.27 1.27)) hide)
-    )
-    (property "Value" "+5V" (id 1) (at 165.1 110.49 0))
-    (property "Footprint" "" (id 2) (at 165.1 115.57 0)
-      (effects (font (size 1.27 1.27)) hide)
-    )
-    (property "Datasheet" "" (id 3) (at 165.1 115.57 0)
-      (effects (font (size 1.27 1.27)) hide)
-    )
-    (pin "1")
-  )
   (sheet_instances
     (path "/" (page "1"))
   )
   (symbol_instances
-    (path "/8aaeb1e4-5a1c-433d-9382-2cc32e56a354"
-      (reference "#PWR01") (unit 1) (value "+5V") (footprint "")
-    )
     (path "/efec6caf-ab5c-4e9e-b71a-caeb1937d304"
       (reference "#PWR02") (unit 1) (value "GND") (footprint "")
     )
-    (path "/f219ead5-5cac-4773-812c-bca3b64657fb"
-      (reference "#PWR03") (unit 1) (value "+5V") (footprint "")
-    )
     (path "/458f86eb-a381-40a0-816e-39a6ea7078c1"
       (reference "#PWR04") (unit 1) (value "GND") (footprint "")
     )
+    (path "/19cb6b6a-fdd0-4db0-8046-677b75254de1"
+      (reference "#PWR0101") (unit 1) (value "+3V3") (footprint "")
+    )
+    (path "/86bb63e4-bce5-4573-ba4a-d78fbe2cc261"
+      (reference "#PWR?") (unit 1) (value "+3V3") (footprint "")
+    )
     (path "/af11a576-d68f-4cdc-8cca-580db2389094"

Commit message: Diode UPdate
Parts:
- D1: footprint Diode_THT:D_T-1_P5.08mm_Horizontal -> Diode_THT:D_DO-41_SOD81_P10.16mm_Horizontal; symbol pspice:DIODE -> Diode:1N4002
Connections:
- net at J1.5, U1.2 (CATHODE): now also D1.2 (A); no longer D1.1 (K)
- net at R1.1, U1.1 (ANODE): now also D1.1 (K); no longer D1.2 (A)

Commit message: Add files via upload
Parts:
- D1: footprint Diode_THT:D_DO-41_SOD81_P10.16mm_Horizontal -> Diode_THT:D_DO-201AD_P15.24mm_Horizontal; symbol Diode:1N4002 -> Diode:1N5404
